Commit message: updates to leg urdf

File: robots/leg_test.urdf.xacro (robot description, xacro)
@@ -1,4 +1,11 @@
-<robot name="reemc"
+<robot name="lobot"
     xmlns:xacro="http://ros.org/wiki/xacro">
+    <xacro:include filename="$(find lobot_description)/urdf/materials.urdf.xacro" />
+    <link name="world" />
+    <joint name="world_joint" type="fixed">
+        <parent link="world" />
+        <child link="base_link" />
+        <origin xyz="0  0 0.6" rpy="0 0 0" />
+    </joint>
     <link name="base_link">
         <inertial>
@@ -17,9 +24,11 @@
             <origin xyz="-0.022 0 0.01" rpy="0 0 0" />
             <geometry>
-                <box size="0.3 0.35 0.14"/>
+                <box size="0.01 0.01 0.01"/>
+                <!-- <box size="0.3 0.35 0.14"/> -->
             </geometry>
         </collision>
     </link>
     <xacro:include filename="$(find lobot_description)/urdf/leg/leg.urdf.xacro" />
+    <!-- <xacro:include filename="$(find lobot_description)/gazebo/gazebo.urdf.xacro" /> -->
     <xacro:lobot_leg name="leg" side="right" reflect="1.0" parent="base_link"/>
     <xacro:lobot_leg name="leg" side="left" reflect="-1.0" parent="base_link"/>

File: urdf/leg/leg.transmission.xacro (robot description, xacro)
@@ -8,6 +8,6 @@
       </actuator>
       <joint name="${name}_${side}_${number}_joint">
-        <hardwareInterface>hardware_interface/PositionJointInterface</hardwareInterface>
-        <!-- <hardwareInterface>hardware_interface/EffortJointInterface</hardwareInterface> -->
+        <!-- <hardwareInterface>hardware_interface/PositionJointInterface</hardwareInterface> -->
+        <hardwareInterface>hardware_interface/EffortJointInterface</hardwareInterface>
       </joint>
     </transmission>

File: urdf/leg/leg.urdf.xacro (robot description, xacro)
@@ -1,3 +1,3 @@
-<?xml version="1.0"?>
+<?xml version="1.0" ?>
 <!--
   Copyright (c) 2011-2012, PAL Robotics, S.L.
@@ -7,6 +7,5 @@
   Creative Commons, 444 Castro Street, Suite 900, Mountain View, California, 94041, USA.
 -->
-<robot name="lobot"
-    xmlns:xacro="http://ros.org/wiki/xacro">
+<robot name="lobot" xmlns:xacro="http://ros.org/wiki/xacro">
     <!--File includes-->
     <xacro:include filename="$(find lobot_description)/urdf/leg/leg.transmission.xacro" />
@@ -18,5 +17,5 @@
     <xacro:property name="leg_eps" value="0.0" />
     <xacro:property name="leg_version" value="0.0" />
-    <xacro:property name="leg_1_joint_max_vel" value="2.74" />
+    <xacro:property name="leg_1_joint_max_vel" value="4" />
     <xacro:property name="leg_2_joint_max_vel" value="${3.94 if leg_version=='v1' else 2.27}" />
     <xacro:property name="leg_3_joint_max_vel" value="${6.0  if leg_version=='v1' else 3.64}" />
@@ -33,46 +32,90 @@
         <link name="leg_${side}_1_link">
             <inertial>
-                <mass value="1.02901"/>
-                <origin xyz="-0.02571 0 0.02557" rpy="0 0 0"/>
-                <inertia ixx="0.00132187534" ixy="0.00000001514" ixz="0.00040022268" iyy="0.0018528617" iyz="0.00000050713" izz="0.00084231334"/>
+                <mass value="1.02901" />
+                <origin xyz="-0.02571 0 0.02557" rpy="0 0 0" />
+                <inertia ixx="0.00132187534" ixy="0.00000001514" ixz="0.00040022268" iyy="0.0018528617" iyz="0.00000050713" izz="0.00084231334" />
             </inertial>
             <visual>
-                <origin rpy="0 0 0" xyz="0 0 0"/>
+                <origin xyz="0 0 -0.03" rpy="0 0 0" />
                 <geometry>
-                    <box size="0.15 0.10 0.20"/>
+                    <box size="0.04 0.10 0.05" />
+                </geometry>
+                <material name="LightGrey" />
+            </visual>
+            <collision>
+                <origin xyz="0 0 0" rpy="0 0 0" />
+                <geometry>
+                    <box size="0.04 0.10 0.05" />
+                </geometry>
+            </collision>
+        </link>
+        <joint name="leg_${side}_1_joint" type="revolute">
+            <origin xyz="0  ${-reflect*0.075} -0.08" rpy="0 0 0" />
+            <axis xyz="1 0 0" />
+            <parent link="${parent}" />
+            <child link="leg_${side}_1_link" />
+            <limit lower="-1.57" upper="1.57" effort="50" velocity="4" />
+        </joint>
+        <link name="leg_${side}_2_link">
+            <inertial>
+                <mass value="0.69621" />
+                <origin xyz="0.00057	${-reflect*0.00881}	-0.01125" rpy="0.0 0.0 0.0" />
+                <inertia ixx="0.0008416476" ixy="-0.00000268743" ixz="0.00000667199" iyy="0.00039794844" iyz="0.00002668971" izz="0.00084196694" />
+            </inertial>
+            <visual>
+                <origin rpy="0 0 0" xyz="0 0 0" />
+                <geometry>
+                    <box size="0.05 0.10 0.05" />
                 </geometry>
                 <material name="LightGrey" />
             </visual>
         </link>
-        <joint name="leg_${side}_1_joint" type="revolute">
-            <origin xyz="0  ${-reflect*0.075} -0.14353" rpy="0 0 0"/>
-            <axis xyz="0 0 1"/>
-            <parent link="${parent}"/>
-            <child link="leg_${side}_1_link"/>
+        <joint name="leg_${side}_2_joint" type="revolute">
+            <origin xyz="0 0 -0.07" rpy="0 0 0" />
+            <axis xyz="0 1 0" />
+            <parent link="leg_${side}_1_link" />
+            <child link="leg_${side}_2_link" />
+            <limit lower="${-22.5*deg_to_rad - reflect*7.5*deg_to_rad}" upper="${22.5*deg_to_rad - reflect*7.5*deg_to_rad}" effort="${leg_2_joint_effort}" velocity="${leg_2_joint_max_vel}" />
+        </joint>
+        <link name="leg_${side}_3_link">
+            <inertial>
+              <mass value="3.97852"/>
+              <origin xyz="0.14784 -0.01646 ${-reflect*0.01793}" rpy="0.0 0 0.0"/>
+              <inertia ixx="0.00507885174" ixy="-0.00034076421" ixz="-0.00225952731" iyy="0.02850097402" iyz="0.00003047874" izz="0.02632392239"/>
+            </inertial>
+           <visual>
+              <origin rpy="0 0 0" xyz="0 0 0"/>
+              <geometry>
+                <box size="0.15 0.10 0.05" />
+              </geometry>
+              <material name="LightGrey" />
+            </visual>
+            <collision>
+              <origin rpy="0 0 0" xyz="0.15 0 ${-reflect*0.015}"/>
+              <geometry>
+                <box size="0.15 0.10 0.20"/>
+              </geometry>
+            </collision>
+          </link>
+          <joint name="leg_${side}_3_joint" type="revolute">
+            <origin xyz="0.06 0 -0.12" rpy="0 0 0" />
+            <axis xyz="0 1 0"/>
+            <parent link="leg_${side}_2_link"/>
+            <child link="leg_${side}_3_link"/>
             <dynamics friction="${leg_friction}" damping="${leg_damping}"/>
-            <limit lower="${-37.5*deg_to_rad + reflect*7.5*deg_to_rad}" upper="${37.5*deg_to_rad + reflect*7.5*deg_to_rad}" effort="${leg_1_joint_effort}" velocity="${leg_1_joint_max_vel}" />
-            <safety_controller k_position="100" k_velocity="100" soft_lower_limit="${-37.5*deg_to_rad + reflect*7.5*deg_to_rad + leg_eps}" soft_upper_limit="${ 37.5*deg_to_rad + reflect*7.5*deg_to_rad - leg_eps}" />
-        </joint>
+            <limit lower="${ -100.0 * deg_to_rad}" upper="${45 * deg_to_rad}" effort="${leg_3_joint_effort}" velocity="${leg_3_joint_max_vel}" />
+            <safety_controller k_position="100"
+                               k_velocity="100"
+                               soft_lower_limit="${-100.0 * deg_to_rad + leg_eps}"
+                               soft_upper_limit="${  45.0 * deg_to_rad - leg_eps}" />
+          </joint>
         <gazebo reference="leg_${side}_1_link">
             <mu1>0.9</mu1>
             <mu2>0.9</mu2>
         </gazebo>
-        <!-- contact model for foot surface -->
-        <!-- <gazebo reference="leg_${side}_6_link">
-            <kp>1000000.0</kp>
-            <kd>100.0</kd>
-            <mu1>1.0</mu1>
-            <mu2>1.0</mu2>
-            <fdir1>0 0 1</fdir1>
-            <maxVel>1.0</maxVel>
-            <minDepth>0.00</minDepth>
-            <implicitSpringDamper>1</implicitSpringDamper>
-        </gazebo> -->
-        <!--force torque sensor -->
-        <!--xacro:reemc_force_torque_sensor name="leg_${side}_6_link" update_rate="100.0"/-->
         <gazebo reference="leg_${side}_1_joint">
             <implicitSpringDamper>1</implicitSpringDamper>
         </gazebo>
-        <!-- <gazebo reference="leg_${side}_2_joint">
+        <gazebo reference="leg_${side}_2_joint">
             <implicitSpringDamper>1</implicitSpringDamper>
         </gazebo>
@@ -80,4 +123,5 @@
             <implicitSpringDamper>1</implicitSpringDamper>
         </gazebo>
+        <!--
         <gazebo reference="leg_${side}_4_joint">
             <implicitSpringDamper>1</implicitSpringDamper>
@@ -91,9 +135,11 @@
         </gazebo> -->
         <xacro:lobot_leg_transmission name="${name}" side="${side}" number="1" reduction="${leg_reduction}" />
-        <!-- <xacro:reemc_leg_simple_transmission name="${name}" side="${side}" number="2" reduction="${leg_reduction}" />
-        <xacro:reemc_leg_simple_transmission name="${name}" side="${side}" number="3" reduction="${leg_reduction}" />
-        <xacro:reemc_leg_simple_transmission name="${name}" side="${side}" number="4" reduction="${leg_reduction}" />
-        <xacro:reemc_leg_simple_transmission name="${name}" side="${side}" number="5" reduction="${leg_reduction}" />
-        <xacro:reemc_leg_simple_transmission name="${name}" side="${side}" number="6" reduction="${leg_reduction}" /> -->
+        <xacro:lobot_leg_transmission name="${name}" side="${side}" number="2" reduction="${leg_reduction}" />
+        <xacro:lobot_leg_transmission name="${name}" side="${side}" number="3" reduction="${leg_reduction}" />
+        <!--
+        <xacro:lobot_leg_simple_transmission name="${name}" side="${side}" number="4" reduction="${leg_reduction}" />
+        <xacro:lobot_leg_simple_transmission name="${name}" side="${side}" number="5" reduction="${leg_reduction}" />
+        <xacro:lobot_leg_simple_transmission name="${name}" side="${side}" number="6" reduction="${leg_reduction}" />
+        -->
     </xacro:macro>
 </robot>
