Commit message: add mass and inertia properties

File: robots/arm_standalone.urdf.xacro (robot description, xacro)
@@ -28,20 +28,20 @@
     </link>
     <joint name="arm_1_joint" type="revolute">
-        <origin xyz="0 0.01 0.052" rpy="0 0 0" />
+        <origin xyz="0 0.01 0.0" rpy="0 0 0" />
         <axis xyz="0 0 1" />
         <parent link="arm_1_link" />
-        <child link="arm_2_interm_link" />
+        <child link="arm_bracket_1" />
         <limit lower="-2.356" upper="2.356" effort="50" velocity="40" />
     </joint>
-    <link name="arm_2_interm_link">
-        <inertial>
-            <mass value="0.00001" />
-            <origin xyz="0 0 0" rpy="0 0 0" />
-            <inertia ixx="0.0" ixy="0.0" ixz="0.0" iyy="0.0" iyz="0.0" izz="0.0" />
-        </inertial>
-        <visual>
-            <origin xyz="0 0 0" rpy="0 0 0" />
-            <geometry>
-                <sphere radius="0.01" />
+    <link name="arm_bracket_1">
+        <inertial>
+            <mass value="0.00658" />
+            <origin xyz="0 0 0.03693" rpy="0 0 0" />
+            <inertia ixx="0.00097149" ixy="0.0" ixz="0.0" iyy="0.00390446" iyz="0.0" izz="0.00346115" />
+        </inertial>
+        <visual>
+            <origin xyz="0 0 0.029" rpy="0 0 0" />
+            <geometry>
+                <box size="0.052 0.025 0.002" />
             </geometry>
             <material name="Green" />
@@ -49,15 +49,16 @@
     </link>
     <joint name="arm_2_joint" type="revolute">
-        <origin xyz="0 0 0" rpy="0 0 0" />
+        <origin xyz="0 0 0.052" rpy="0 0 0" />
         <axis xyz="1 0 0" />
-        <parent link="arm_2_interm_link" />
+        <parent link="arm_bracket_1" />
         <child link="arm_2_link" />
         <limit lower="-2.356" upper="2.356" effort="50" velocity="40" />
     </joint>
+    <!-- arm_2_link = motor2 -->
     <link name="arm_2_link">
         <inertial>
-            <mass value="0.06" />
-            <origin xyz="0 -0.01 0" rpy="0 0 0" />
-            <inertia ixx="0.0" ixy="0.0" ixz="0.0" iyy="0.0" iyz="0.0" izz="0.0" />
+            <mass value="0.0618" />
+            <origin xyz="0.0005 -0.01505 0" rpy="0 0 0" />
+            <inertia ixx="0.00703304" ixy="-0.00250174" ixz="0.0" iyy="0.00793603" iyz="0.0" izz="0.01230371" />
         </inertial>
         <visual>
@@ -69,11 +70,36 @@
         </visual>
         <collision>
-            <origin rpy="0 0 0" xyz="0 0 0" />
-            <geometry>
-                <box size="0.04 0.04 0.02" />
-            </geometry>
-            <material name="LightGrey" />
-        </collision>
-    </link>
+            <origin xyz="0 -0.01 0" rpy="0 0 0" />
+            <geometry>
+                <box size="0.04 0.04 0.02" />
+            </geometry>
+        </collision>
+    </link>
+    <!-- arm_bracket_2 = Asm_WeldedBracket -->
+    <link name="arm_bracket_2">
+        <inertial>
+            <mass value="0.01175" />
+            <origin xyz="0 -0.0029 0" rpy="0 0 0" />
+            <inertia ixx="0.00229954" ixy="0.0" ixz="0.0" iyy="0.00519619" iyz="0.0" izz="0.00648306" />
+        </inertial>
+        <visual>
+            <origin xyz="0 0 0" rpy="0 0 0" />
+            <geometry>
+                <box size="0.055 0.002 0.025" />
+            </geometry>
+            <material name="Green" />
+        </visual>
+        <collision>
+            <origin xyz="0 0 0" rpy="0 0 0" />
+            <geometry>
+                <box size="0.055 0.002 0.025" />
+            </geometry>
+        </collision>
+    </link>
+    <joint name="arm_bracket_2_joint" type="fixed">
+        <parent link="arm_2_link" />
+        <child link="arm_bracket_2" />
+        <origin xyz="0 -0.03653 0" rpy="0 0 0" />
+    </joint>
     <joint name="arm_3_joint" type="revolute">
         <origin xyz="0 -0.06 0" rpy="0 0 0" />
@@ -83,9 +109,10 @@
         <limit lower="-2.356" upper="2.356" effort="50" velocity="40" />
     </joint>
+    <!-- arm_3_link = motor3 -->
     <link name="arm_3_link">
         <inertial>
-            <mass value="0.06" />
-            <origin xyz="0 -0.01 0" rpy="0 0 0" />
-            <inertia ixx="0.0" ixy="0.0" ixz="0.0" iyy="0.0" iyz="0.0" izz="0.0" />
+            <mass value="0.0618" />
+            <origin xyz="0.0005 -0.01505 0" rpy="0 0 0" />
+            <inertia ixx="0.00703304" ixy="-0.00250174" ixz="0.0" iyy="0.00793603" iyz="0.0" izz="0.01230371" />
         </inertial>
         <visual>
@@ -97,11 +124,11 @@
         </visual>
         <collision>
-            <origin rpy="0 0 0" xyz="0 0 0" />
-            <geometry>
-                <box size="0.04 0.04 0.02" />
-            </geometry>
-            <material name="LightGrey" />
-        </collision>
-    </link>
+            <origin xyz="0 -0.01 0" rpy="0 0 0" />
+            <geometry>
+                <box size="0.04 0.04 0.02" />
+            </geometry>
+        </collision>
+    </link>
+    <!-- The entire grippper mass property is put on the first link -->
     <joint name="grip_joint_1" type="fixed">
         <parent link="arm_3_link" />
@@ -111,7 +138,7 @@
     <link name="grip_link_1">
         <inertial>
-            <mass value="0.005" />
-            <origin xyz="0 0 0" rpy="0 0 0" />
-            <inertia ixx="0.0" ixy="0.0" ixz="0.0" iyy="0.0" iyz="0.0" izz="0.0" />
+            <mass value="0.01023" />
+            <origin xyz="0 -0.05355 0" rpy="0 0 0" />
+            <inertia ixx="0.00443574" ixy="0.0" ixz="0.0" iyy="0.00287052" iyz="0.00000684" izz="0.00651523" />
         </inertial>
         <visual>
@@ -123,9 +150,8 @@
         </visual>
         <collision>
-            <origin xyz="0 -0.01 0" rpy="0 0 0" />
-            <geometry>
-                <box size="0.055 0.04 0.001" />
-            </geometry>
-            <material name="White" />
+            <origin xyz="0 0 0" rpy="0 0 0" />
+            <geometry>
+                <box size="0.04 0.055 0.001" />
+            </geometry>
         </collision>
     </link>
@@ -149,9 +175,8 @@
         </visual>
         <collision>
-            <origin xyz="0 -0.01 0" rpy="0 0 0" />
-            <geometry>
-                <box size="0.055 0.04 0.001" />
-            </geometry>
-            <material name="White" />
+            <origin xyz="0 0 0" rpy="0.785398 0 0" />
+            <geometry>
+                <box size="0.04 0.017 0.001" />
+            </geometry>
         </collision>
     </link>
@@ -175,7 +200,7 @@
         </visual>
         <collision>
-            <origin xyz="0 -0.01 0" rpy="0 0 0" />
-            <geometry>
-                <box size="0.055 0.04 0.001" />
+            <origin xyz="0 0 0" rpy="0 0 0" />
+            <geometry>
+                <box size="0.04 0.001 0.007" />
             </geometry>
             <material name="White" />

Commit message: add gazebo plugins

File: robots/arm_standalone.urdf.xacro (robot description, xacro)
@@ -1,4 +1,6 @@
 <robot name="lobot" xmlns:xacro="http://ros.org/wiki/xacro">
     <xacro:include filename="$(find lobot_description)/urdf/materials.urdf.xacro" />
+    <xacro:include filename="$(find lobot_description)/gazebo/gazebo_arm.urdf.xacro" />
+    <xacro:gazebo_macro robot="arm_standalone" control_update_rate="100" status_update_rate="500" />
     <link name="world" />
     <joint name="world_joint" type="fixed">
@@ -47,4 +49,10 @@
             <material name="Green" />
         </visual>
+        <collision>
+            <origin xyz="0 0 0.029" rpy="0 0 0" />
+            <geometry>
+                <box size="0.052 0.025 0.002" />
+            </geometry>
+        </collision>
     </link>
     <joint name="arm_2_joint" type="revolute">
@@ -204,5 +212,4 @@
                 <box size="0.04 0.001 0.007" />
             </geometry>
-            <material name="White" />
         </collision>
     </link>

Commit message: update limits

File: robots/arm_standalone.urdf.xacro (robot description, xacro)
@@ -34,5 +34,5 @@
         <parent link="arm_1_link" />
         <child link="arm_bracket_1" />
-        <limit lower="-2.356" upper="2.356" effort="50" velocity="40" />
+        <limit lower="-2.356" upper="2.356" effort="20" velocity="10" />
     </joint>
     <link name="arm_bracket_1">
@@ -61,5 +61,5 @@
         <parent link="arm_bracket_1" />
         <child link="arm_2_link" />
-        <limit lower="-2.356" upper="2.356" effort="50" velocity="40" />
+        <limit lower="-1.570796" upper="1.570796" effort="20" velocity="20" />
     </joint>
     <!-- arm_2_link = motor2 -->
@@ -115,5 +115,5 @@
         <parent link="arm_2_link" />
         <child link="arm_3_link" />
-        <limit lower="-2.356" upper="2.356" effort="50" velocity="40" />
+        <limit lower="-1.570796" upper="1.570796" effort="10" velocity="10" />
     </joint>
     <!-- arm_3_link = motor3 -->
