Commit message: initial prototype

File: gazebo/gazebo.urdf.xacro (robot description, xacro)
@@ -1,92 +1,24 @@
-<?xml version="1.0"?>
-<!--
-  Copyright (c) 2011, PAL Robotics, S.L.
-  All rights reserved.
-  This work is licensed under the Creative Commons Attribution-NonCommercial-NoDerivs 3.0 Unported License.
-  To view a copy of this license, visit http://creativecommons.org/licenses/by-nc-nd/3.0/ or send a letter to
-  Creative Commons, 444 Castro Street, Suite 900, Mountain View, California, 94041, USA.
--->
-<robot name="lobot">
+<?xml version="1.0" ?>
+<robot xmlns:xacro="http://ros.org/wiki/xacro" name="lobot">
   <gazebo>
-    <plugin filename="libgazebo_ros_control.so" name="gazebo_ros_control">
-      <robotNamespace>/lobot</robotNamespace>
-      <robotSimType>gazebo_ros_control/DefaultRobotHWSim</robotSimType>
-    </plugin>
-    <plugin filename="libgazebo_ros_p3d.so" name="gazebo_ros_p3d">
-      <bodyName>base_link</bodyName>
-      <topicName>ground_truth_odom</topicName>
-      <alwaysOn>true</alwaysOn>
-      <updateRate>100.0</updateRate>
+    <plugin filename="libmy_joint_state_publisher.so" name="my_joint_state_publisher">
+      <robot_name>lobot</robot_name>
+      <update_rate>500</update_rate>
     </plugin>
   </gazebo>
   <gazebo>
-    <plugin filename="libgazebo_ros_force.so" name="gazebo_ros_force">
-      <bodyName>base_link</bodyName>
-      <topicName>base_link_wrench</topicName>
+    <plugin filename="librobot_plugin.so" name="robot_plugin_lobot">
+      <robot_name>lobot</robot_name>
+      <update_rate>1000</update_rate>
     </plugin>
   </gazebo>
-  <gazebo>
-    <plugin filename="libgazebo_world_odometry.so" name="gazebo_ros_odometry">
-      <frameName>base_link</frameName>
-      <topicName>floating_base_pose_simulated</topicName>
-    </plugin>
-  </gazebo>
-  <gazebo reference="imu_link">
-    <!-- this is expected to be reparented to pelvis with appropriate offset
-         when imu_link is reduced by fixed joint reduction -->
-    <!-- todo: this is working with gazebo 1.4, need to write a unit test -->
-    <sensor name="imu_sensor" type="imu">
-      <always_on>1</always_on>
-      <update_rate>1000.0</update_rate>
-      <imu>
-        <noise>
-          <type>gaussian</type>
-          <!-- Noise parameters from Boston Dynamics
-               (http://gazebosim.org/wiki/Sensor_noise):
-                 rates (rad/s): mean=0, stddev=2e-4
-                 accels (m/s/s): mean=0, stddev=1.7e-2
-                 rate bias (rad/s): 5e-6 - 1e-5
-                 accel bias (m/s/s): 1e-1
-               Experimentally, simulation provide rates with noise of
-               about 1e-3 rad/s and accels with noise of about 1e-1 m/s/s.
-               So we don't expect to see the noise unless number of inner iterations
-               are increased.
-               We will add bias.  In this model, bias is sampled once for rates
-               and once for accels at startup; the sign (negative or positive)
-               of each bias is then switched with equal probability.  Thereafter,
-               the biases are fixed additive offsets.  We choose
-               bias means and stddevs to produce biases close to the provided
-               data. -->
-          <rate>
-            <mean>0.0</mean>
-            <stddev>2e-4</stddev>
-            <bias_mean>0.0000075</bias_mean>
-            <bias_stddev>0.0000008</bias_stddev>
-          </rate>
-          <accel>
-            <mean>0.0</mean>
-            <stddev>1.7e-2</stddev>
-            <bias_mean>0.1</bias_mean>
-            <bias_stddev>0.001</bias_stddev>
-          </accel>
-        </noise>
-      </imu>
+  <gazebo reference="IMU_link">
+    <sensor type="imu" name="IMU_lobot">
+      <always_on>true</always_on>
+      <update_rate>10.0</update_rate>
+      <plugin filename="libgazebo_ros_imu_sensor.so" name="lobot_IMU_controller"></plugin>
     </sensor>
   </gazebo>
-  <gazebo reference="r_foot">
-    <mu1>0.9</mu1>
-    <mu2>0.9</mu2>
-    <fdir1>1 0 0</fdir1>
-    <maxVel>1.0</maxVel>
-    <minDepth>0.003</minDepth>
-  </gazebo>
-  <gazebo reference="l_foot">
-    <mu1>0.9</mu1>
-    <mu2>0.9</mu2>
-    <fdir1>1 0 0</fdir1>
-    <maxVel>1.0</maxVel>
-    <minDepth>0.003</minDepth>
-  </gazebo>
   <!-- define global properties -->
-  <property name="M_PI" value="3.1415926535897931" />
+  <xacro:property name="M_PI" value="3.1415926535897931" />
 </robot>

File: urdf/leg/leg.urdf.xacro (robot description, xacro)
@@ -1,9 +1,7 @@
 <?xml version="1.0" ?>
 <!--
-  Copyright (c) 2011-2012, PAL Robotics, S.L.
+  Author: Poh Zhi-Ee (zhiee.poh@httechnology.com)
+  Copyright (c) 2019, SIW Manufacturing Sdn. Bhd.
   All rights reserved.
-  This work is licensed under the Creative Commons Attribution-NonCommercial-NoDerivs 3.0 Unported License.
-  To view a copy of this license, visit http://creativecommons.org/licenses/by-nc-nd/3.0/ or send a letter to
-  Creative Commons, 444 Castro Street, Suite 900, Mountain View, California, 94041, USA.
 -->
 <robot name="lobot" xmlns:xacro="http://ros.org/wiki/xacro">
@@ -32,82 +30,166 @@
         <link name="leg_${side}_1_link">
             <inertial>
-                <mass value="1.02901" />
-                <origin xyz="-0.02571 0 0.02557" rpy="0 0 0" />
+                <mass value="0.02901" />
+                <origin xyz="0 0 0" rpy="0.0 0.0 0.0" />
                 <inertia ixx="0.00132187534" ixy="0.00000001514" ixz="0.00040022268" iyy="0.0018528617" iyz="0.00000050713" izz="0.00084231334" />
             </inertial>
             <visual>
-                <origin xyz="0 0 -0.03" rpy="0 0 0" />
-                <geometry>
-                    <box size="0.04 0.10 0.05" />
-                </geometry>
-                <material name="LightGrey" />
-            </visual>
-            <collision>
-                <origin xyz="0 0 0" rpy="0 0 0" />
-                <geometry>
-                    <box size="0.04 0.10 0.05" />
+                <origin rpy="0 ${90*deg_to_rad} 0" xyz="0 0 0" />
+                <geometry>
+                    <cylinder radius="0.01" length="0.02" />
+                </geometry>
+                <material name="LightGrey" />
+            </visual>
+            <collision>
+                <origin rpy="0 ${90*deg_to_rad} 0" xyz="0 0 0" />
+                <geometry>
+                    <cylinder radius="0.01" length="0.02" />
                 </geometry>
             </collision>
         </link>
         <joint name="leg_${side}_1_joint" type="revolute">
-            <origin xyz="0  ${-reflect*0.075} -0.08" rpy="0 0 0" />
+            <origin xyz="0  ${-reflect*0.0315} -0.0475" rpy="0 0 0" />
             <axis xyz="1 0 0" />
             <parent link="${parent}" />
             <child link="leg_${side}_1_link" />
-            <limit lower="-1.57" upper="1.57" effort="50" velocity="4" />
+            <limit lower="-1.2" upper="1.2" effort="50" velocity="4"/>
         </joint>
         <link name="leg_${side}_2_link">
             <inertial>
-                <mass value="0.69621" />
-                <origin xyz="0.00057	${-reflect*0.00881}	-0.01125" rpy="0.0 0.0 0.0" />
-                <inertia ixx="0.0008416476" ixy="-0.00000268743" ixz="0.00000667199" iyy="0.00039794844" iyz="0.00002668971" izz="0.00084196694" />
-            </inertial>
-            <visual>
-                <origin rpy="0 0 0" xyz="0 0 0" />
-                <geometry>
-                    <box size="0.05 0.10 0.05" />
-                </geometry>
-                <material name="LightGrey" />
-            </visual>
+                <mass value="0.069621" />
+                <origin xyz="0 0 0" rpy="0.0 0.0 0.0" />
+                <inertia ixx="0.0008416476" ixy="-0.00000268743" ixz="0.00000667199" iyy="0.00039794844" iyz="0.00002668971" izz="0.00084196694" />
+            </inertial>
+            <visual>
+                    <origin rpy="0 ${26.565*deg_to_rad} 0" xyz="0.02 0 0" />
+                <geometry>
+                    <!-- <cylinder radius="0.01" length="0.02" /> -->
+                    <box size="0.02 0.04 0.02" />
+                </geometry>
+                <material name="LightGrey" />
+            </visual>
+            <collision>
+                <origin rpy="0 ${26.565*deg_to_rad} 0" xyz="0.02 0 0" />
+                <geometry>
+                    <!-- <cylinder radius="0.01" length="0.02" /> -->
+                    <box size="0.03 0.03 0.02" />
+                </geometry>
+            </collision>
         </link>
         <joint name="leg_${side}_2_joint" type="revolute">
-            <origin xyz="0 0 -0.07" rpy="0 0 0" />
+            <origin xyz="0 0 -0.04707" rpy="0 0 0" />
             <axis xyz="0 1 0" />
             <parent link="leg_${side}_1_link" />
             <child link="leg_${side}_2_link" />
-            <limit lower="${-22.5*deg_to_rad - reflect*7.5*deg_to_rad}" upper="${22.5*deg_to_rad - reflect*7.5*deg_to_rad}" effort="${leg_2_joint_effort}" velocity="${leg_2_joint_max_vel}" />
+            <limit lower="-1.2" upper="1.2" effort="50" velocity="4"/>
+        </joint>
+        <link name="leg_${side}_3a_link">
+            <inertial>
+                <mass value="0.04" />
+                <origin xyz="0 0 0" rpy="0.0 0.0 0.0" />
+                <inertia ixx="0.0008416476" ixy="-0.00000268743" ixz="0.00000667199" iyy="0.00039794844" iyz="0.00002668971" izz="0.00084196694" />
+            </inertial>
+            <visual>
+                <origin rpy="0 0 0" xyz="0 0 0.004" />
+                <geometry>
+                    <box size="0.02 0.04 0.025" />
+                </geometry>
+                <material name="LightGrey" />
+            </visual>
+            <collision>
+                <origin rpy="0 0 0" xyz="0 0 0.004" />
+                <geometry>
+                    <box size="0.02 0.04 0.025" />
+                </geometry>
+            </collision>
+        </link>
+        <joint name="leg_${side}_3a_joint" type="fixed">
+            <origin xyz="0.04104 0 -0.020" rpy="0 0 0" />
+            <parent link="leg_${side}_2_link" />
+            <child link="leg_${side}_3a_link" />
         </joint>
         <link name="leg_${side}_3_link">
             <inertial>
-              <mass value="3.97852"/>
-              <origin xyz="0.14784 -0.01646 ${-reflect*0.01793}" rpy="0.0 0 0.0"/>
-              <inertia ixx="0.00507885174" ixy="-0.00034076421" ixz="-0.00225952731" iyy="0.02850097402" iyz="0.00003047874" izz="0.02632392239"/>
-            </inertial>
-           <visual>
-              <origin rpy="0 0 0" xyz="0 0 0"/>
-              <geometry>
-                <box size="0.15 0.10 0.05" />
-              </geometry>
-              <material name="LightGrey" />
-            </visual>
-            <collision>
-              <origin rpy="0 0 0" xyz="0.15 0 ${-reflect*0.015}"/>
-              <geometry>
-                <box size="0.15 0.10 0.20"/>
-              </geometry>
-            </collision>
-          </link>
-          <joint name="leg_${side}_3_joint" type="revolute">
-            <origin xyz="0.06 0 -0.12" rpy="0 0 0" />
-            <axis xyz="0 1 0"/>
-            <parent link="leg_${side}_2_link"/>
-            <child link="leg_${side}_3_link"/>
-            <dynamics friction="${leg_friction}" damping="${leg_damping}"/>
-            <limit lower="${ -100.0 * deg_to_rad}" upper="${45 * deg_to_rad}" effort="${leg_3_joint_effort}" velocity="${leg_3_joint_max_vel}" />
-            <safety_controller k_position="100"
-                               k_velocity="100"
-                               soft_lower_limit="${-100.0 * deg_to_rad + leg_eps}"
-                               soft_upper_limit="${  45.0 * deg_to_rad - leg_eps}" />
-          </joint>
+                <mass value="0.05" />
+                <origin xyz="0 0 0" rpy="0.0 0.0 0.0" />
+                <inertia ixx="0.0008416476" ixy="-0.00000268743" ixz="0.00000667199" iyy="0.00039794844" iyz="0.00002668971" izz="0.00084196694" />
+            </inertial>
+            <visual>
+                <origin rpy="0 0 0" xyz="0 0 -0.02" />
+                <geometry>
+                    <box size="0.02 0.04 0.04" />
+                </geometry>
+                <material name="LightGrey" />
+            </visual>
+            <collision>
+                <origin rpy="0 0 0" xyz="0 0 -0.02" />
+                <geometry>
+                    <box size="0.02 0.04 0.04" />
+                </geometry>
+            </collision>
+        </link>
+        <joint name="leg_${side}_3_joint" type="revolute">
+            <origin xyz="0 0 -0.02477" rpy="0 0 0" />
+            <axis xyz="0 1 0" />
+            <parent link="leg_${side}_3a_link" />
+            <child link="leg_${side}_3_link" />
+            <limit lower="-1.2" upper="1.2" effort="50" velocity="4"/>
+        </joint>
+        <link name="leg_${side}_4_link">
+            <inertial>
+                <mass value="0.06" />
+                <origin xyz="0 0 0" rpy="0.0 0.0 0.0" />
+                <inertia ixx="0.0008416476" ixy="-0.00000268743" ixz="0.00000667199" iyy="0.00039794844" iyz="0.00002668971" izz="0.00084196694" />
+            </inertial>
+            <visual>
+                <origin rpy="${90*deg_to_rad} 0 0" xyz="0 0 0" />
+                <geometry>
+                    <cylinder radius="0.01" length="0.02" />
+                </geometry>
+                <material name="LightGrey" />
+            </visual>
+            <collision>
+                <origin rpy="${90*deg_to_rad} 0 0" xyz="0 0 0" />
+                <geometry>
+                    <cylinder radius="0.01" length="0.02" />
+                </geometry>
+            </collision>
+        </link>
+        <joint name="leg_${side}_4_joint" type="revolute">
+            <origin xyz="0 0 -0.05856" rpy="0 0 0" />
+            <axis xyz="0 1 0" />
+            <parent link="leg_${side}_3_link" />
+            <child link="leg_${side}_4_link" />
+            <dynamics friction="${leg_friction}" damping="${leg_damping}" />
+            <limit lower="-1.2" upper="1.2" effort="50" velocity="4"/>
+        </joint>
+        <link name="leg_${side}_5_link">
+            <inertial>
+                <mass value="0.05" />
+                <origin xyz="0 0 0" rpy="0.0 0.0 0.0" />
+                <inertia ixx="0.0008416476" ixy="-0.00000268743" ixz="0.00000667199" iyy="0.00039794844" iyz="0.00002668971" izz="0.00084196694" />
+            </inertial>
+            <visual>
+                <origin rpy="0 0 0" xyz="0 0 -0.005" />
+                <geometry>
+                    <!-- <cylinder radius="0.01" length="0.02" /> -->
+                    <box size="0.095 0.07 0.01" />
+                </geometry>
+                <material name="LightGrey" />
+            </visual>
+            <collision>
+                <origin rpy="0 0 0" xyz="0 0 -0.005" />
+                <geometry>
+                    <box size="0.095 0.07 0.01" />
+                </geometry>
+            </collision>
+        </link>
+        <joint name="leg_${side}_5_joint" type="revolute">
+            <origin xyz="0 0 -0.04707" rpy="0 0 0" />
+            <axis xyz="1 0 0" />
+            <parent link="leg_${side}_4_link" />
+            <child link="leg_${side}_5_link" />
+            <limit lower="-1.2" upper="1.2" effort="50" velocity="4"/>
+        </joint>
         <gazebo reference="leg_${side}_1_link">
             <mu1>0.9</mu1>
@@ -123,8 +205,8 @@
             <implicitSpringDamper>1</implicitSpringDamper>
         </gazebo>
+        <gazebo reference="leg_${side}_4_joint">
+            <implicitSpringDamper>1</implicitSpringDamper>
+        </gazebo>
         <!--
-        <gazebo reference="leg_${side}_4_joint">
-            <implicitSpringDamper>1</implicitSpringDamper>
-        </gazebo>
         <gazebo reference="leg_${side}_5_joint">
             <implicitSpringDamper>1</implicitSpringDamper>
@@ -137,6 +219,7 @@
         <xacro:lobot_leg_transmission name="${name}" side="${side}" number="2" reduction="${leg_reduction}" />
         <xacro:lobot_leg_transmission name="${name}" side="${side}" number="3" reduction="${leg_reduction}" />
+        <xacro:lobot_leg_transmission name="${name}" side="${side}" number="4" reduction="${leg_reduction}" />
+        <xacro:lobot_leg_transmission name="${name}" side="${side}" number="5" reduction="${leg_reduction}" />
         <!--
-        <xacro:lobot_leg_simple_transmission name="${name}" side="${side}" number="4" reduction="${leg_reduction}" />
         <xacro:lobot_leg_simple_transmission name="${name}" side="${side}" number="5" reduction="${leg_reduction}" />
         <xacro:lobot_leg_simple_transmission name="${name}" side="${side}" number="6" reduction="${leg_reduction}" />
