Commit message: update velocity limits

File: urdf/arm/arm.urdf.xacro (robot description, xacro)
@@ -36,5 +36,5 @@
             <parent link="${parent}" />
             <child link="arm_${side}_1_link" />
-            <limit lower="-1.57" upper="1.57" effort="50" velocity="4" />
+            <limit lower="-1.57" upper="1.57" effort="50" velocity="40" />
         </joint>
         <link name="arm_${side}_2_link">
@@ -63,5 +63,5 @@
             <parent link="arm_${side}_1_link" />
             <child link="arm_${side}_2_link" />
-            <limit lower="${-90*deg_to_rad}" upper="${90*deg_to_rad}" effort="50" velocity="4" />
+            <limit lower="${-90*deg_to_rad}" upper="${90*deg_to_rad}" effort="50" velocity="40" />
         </joint>
         <link name="arm_${side}_3_link">
@@ -90,5 +90,5 @@
             <parent link="arm_${side}_2_link" />
             <child link="arm_${side}_3_link" />
-            <limit lower="${-90*deg_to_rad}" upper="${90*deg_to_rad}" effort="50" velocity="4" />
+            <limit lower="${-90*deg_to_rad}" upper="${90*deg_to_rad}" effort="50" velocity="40" />
         </joint>
         <!-- Gripper fixed link-->

File: urdf/leg/leg.urdf.xacro (robot description, xacro)
@@ -53,5 +53,5 @@
             <parent link="${parent}" />
             <child link="leg_${side}_1_link" />
-            <limit lower="-1.2" upper="1.2" effort="50" velocity="4"/>
+            <limit lower="-1.2" upper="1.2" effort="50" velocity="40"/>
         </joint>
         <link name="leg_${side}_2_link">
@@ -72,6 +72,5 @@
                 <origin rpy="0 ${26.565*deg_to_rad} 0" xyz="0.02 0 0" />
                 <geometry>
-                    <!-- <cylinder radius="0.01" length="0.02" /> -->
-                    <box size="0.03 0.03 0.02" />
+                    <box size="0.02 0.04 0.02" />
                 </geometry>
             </collision>
@@ -82,5 +81,5 @@
             <parent link="leg_${side}_1_link" />
             <child link="leg_${side}_2_link" />
-            <limit lower="-1.2" upper="1.2" effort="50" velocity="4"/>
+            <limit lower="-1.2" upper="1.2" effort="50" velocity="40"/>
         </joint>
         <link name="leg_${side}_3a_link">
@@ -134,5 +133,5 @@
             <parent link="leg_${side}_3a_link" />
             <child link="leg_${side}_3_link" />
-            <limit lower="-1.2" upper="1.2" effort="50" velocity="4"/>
+            <limit lower="-1.2" upper="1.2" effort="50" velocity="40"/>
         </joint>
         <link name="leg_${side}_4_link">
@@ -162,5 +161,5 @@
             <child link="leg_${side}_4_link" />
             <dynamics friction="${leg_friction}" damping="${leg_damping}" />
-            <limit lower="-1.2" upper="1.2" effort="50" velocity="4"/>
+            <limit lower="-1.2" upper="1.2" effort="50" velocity="40"/>
         </joint>
         <link name="leg_${side}_5_link">
@@ -190,5 +189,5 @@
             <parent link="leg_${side}_4_link" />
             <child link="leg_${side}_5_link" />
-            <limit lower="-1.2" upper="1.2" effort="50" velocity="4"/>
+            <limit lower="-1.2" upper="1.2" effort="50" velocity="40"/>
         </joint>
         <gazebo reference="leg_${side}_1_link">
